File: MotionSensor/MotionSensor.kicad_sch (KiCad schematic)
At the start: 0 parts

Commit message: b
Parts:
- added C1, C2, C3: 0.1uF, Capacitor_SMD:C_0603_1608Metric_Pad1.08x0.95mm_HandSolder, symbol Device:C
- added D1, D2, D3: SK6812MINI-E, FS:SK6812MINI-E_fixed, symbol Light:SK6812MINI-E
- added J1: SSD1306 Display, FS:SSD1306-0.91-OLED-4pin-128x32, symbol Connector:Conn_01x04_Pin
- added SW1, SW2, SW3: TL3301AF160QG, FS:TL3301_A_G_EWI, symbol Button:TL3301AF160QG
- added TP1, TP2, TP3, TP4, TP5, TP6: TestPoint, TestPoint:TestPoint_Pad_2.0x2.0mm, symbol Connector:TestPoint
- added U1: XIAO-ESP32-C6, xiao_series:XIAO-ESP32-C6-DIP, symbol OPL Library:XIAO_ESP32-C6-DIP
- added U2: XIAO 24GHZ MMWAVE SENSOR, FS:XIAO-14P-Add-On, symbol Motion Sensor:XIAO-Add-On
Connections:
- new net: D1.2 (DOUT), D2.4 (DIN)
- new net: D2.2 (DOUT), D3.4 (DIN)
- new net +3V3: C1.1, C2.1, C3.1, D1.1 (VDD), D2.1 (VDD), D3.1 (VDD), J1.2 (Pin_2), TP2.1, U1.12 (3V3), U2.3 (3V3)
- new net D0: SW1.1, SW1.2, U1.1 (GPIO0/A0/D0)
- new net D1: SW2.1, SW2.2, U1.2 (GPIO1/A1/D1)
- new net D2: SW3.1, SW3.2, U1.3 (GPIO2/A2/D2)
- new net D3: D1.4 (DIN), U1.4 (GPIO21/D3)
- new net GND: C1.2, C2.2, C3.2, D1.3 (VSS), D2.3 (VSS), D3.3 (VSS), J1.1 (Pin_1), SW1.3, SW1.4, SW2.3, SW2.4, SW3.3, SW3.4, TP1.1, U1.13 (GND), U2.2 (GND)
- new net RX-TX: TP5.1, U1.8 (GPIO17/D7/RX), U2.12 (TX)
- new net SCL: J1.3 (Pin_3), TP3.1, U1.6 (GPIO23/D5/SCL)
- new net SDA: J1.4 (Pin_4), TP4.1, U1.5 (GPIO22/D4/SDA)
- new net TX-RX: TP6.1, U1.7 (GPIO16/D6/TX), U2.11 (RX)
- no-connect marks 0 -> 15
Other:
- note added: "BUTTONS"
- note added: "Connectors"
- note added: "LEDS"
- note added: "MCU"
- note added: "SENSOR"
- company: (none) -> Created by Knox E.
- title: (none) -> Matter MMWAVE Motion Sensor Board

Commit message: C
Parts:
- removed C3: 0.1uF, Capacitor_SMD:C_0603_1608Metric_Pad1.08x0.95mm_HandSolder, symbol Device:C
- removed D3: SK6812MINI-E, FS:SK6812MINI-E_fixed, symbol Light:SK6812MINI-E
- removed SW3: TL3301AF160QG, FS:TL3301_A_G_EWI, symbol Button:TL3301AF160QG
- added H1, H2, H3, H4: M2, MountingHole:MountingHole_2.2mm_M2_Pad, symbol Mechanical:MountingHole_Pad
Connections:
- net GND: now also H1.1, H2.1, H3.1, H4.1
- net D0 renamed 0
- net D1 renamed 1
- net D2: no longer names the net of U1.3 (GPIO2/A2/D2)
- net D3 renamed 3
- no-connect marks 15 -> 16
Other:
- note added: "MHs"
- moved on the sheet: SW1, SW2
